File: urban-power-dist-v2/output.kicad_sch (KiCad schematic)
At the start: 4 parts, among them J1 12V_IN

Commit message: With hierarchical sheets
Parts:
- removed D1: TVS_DIODE, Diode_SMD:Nexperia_DSN1608-2_1.6x0.8mm, symbol Diode:PTVS12VZ1USK
- removed D2: LED, LED_SMD:LED_0603_1608Metric_Pad1.05x0.95mm_HandSolder, symbol Device:LED
- removed J1: 12V_IN, ATF13-2P-BM03:ATF132PBM03, symbol Connector:Conn_01x02_Socket
- removed R1: 9.45K, Resistor_SMD:R_1206_3216Metric_Pad1.30x1.75mm_HandSolder, symbol Device:R_US
- added D6: LED, LED_SMD:LED_0603_1608Metric_Pad1.05x0.95mm_HandSolder, symbol Device:LED
- added F4: FUSE, Fuse:Fuseholder_Blade_Mini_Keystone_3568, symbol Device:Fuse
- added J8: TEST_PT, Connector_PinHeader_2.54mm:PinHeader_1x03_P2.54mm_Vertical, symbol Connector:Conn_01x03_Pin
- added J9: OUT, ATF13-2P-BM03:ATF132PBM03, symbol Connector:Conn_01x02_Socket
- added R8: 0.01R, Resistor_SMD:R_0805_2012Metric_Pad1.20x1.40mm_HandSolder, symbol Device:R_US
- added R9: 9.45K, Resistor_SMD:R_1206_3216Metric_Pad1.30x1.75mm_HandSolder, symbol Device:R_US
Connections:
- net +12V: now also F4.1
- net GND: now also D6.1 (K), J8.3 (Pin_3), J9.2 (Pin_2)
- new net: F4.2, J8.1 (Pin_1), R8.1
- new net: J8.2 (Pin_2), J9.1 (Pin_1), R8.2, R9.2
- new net: D6.2 (A), R9.1
Other:
- removed sheet FRONT_ACC1
- removed sheet REAR_ACC1
- removed sheet TEL_ACC1
- note removed: "12 V Input"
- note removed: "12 V Outputs"

Commit message: pcb layout
Parts:
- renumbered D6 to D3, F4 to F1, J9 to J2, J8 to J5, R9 to R2, R8 to R5
Changed lines of the file:
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@@
 		(on_board yes)
 		(dnp no)
-		(property "Reference" "J8"
+		(property "Reference" "J5"
 			(at 121.666 108.204 0)
 			(effects
@@
 			(project "urban-power-dist-v2"
 				(path "/5f9a1ba6-34f0-4af5-b9a9-ffcd8ae2cc01/261ee563-a4e4-4d31-ad5c-99d3e1f31c1d"
-					(reference "J8")
-					(unit 1)
-				)
-				(path "/5f9a1ba6-34f0-4af5-b9a9-ffcd8ae2cc01/b95fc682-bda1-44b2-bae0-b04d00e2d08a"
-					(reference "J2")
-					(unit 1)
-				)
-				(path "/5f9a1ba6-34f0-4af5-b9a9-ffcd8ae2cc01/da044d78-69ae-4295-a410-101a45713a38"
-					(reference "J10")
+					(reference "J5")
+					(unit 1)
+				)
+				(path "/5f9a1ba6-34f0-4af5-b9a9-ffcd8ae2cc01/b95fc682-bda1-44b2-bae0-b04d00e2d08a"
+					(reference "J6")
+					(unit 1)
+				)
+				(path "/5f9a1ba6-34f0-4af5-b9a9-ffcd8ae2cc01/da044d78-69ae-4295-a410-101a45713a38"
+					(reference "J7")
 					(unit 1)
 				)
@@
 		(dnp no)
 		(fields_autoplaced yes)
-		(property "Reference" "R8"
+		(property "Reference" "R5"
 			(at 140.97 92.71 90)
 			(effects
@@
 			(project "urban-power-dist-v2"
 				(path "/5f9a1ba6-34f0-4af5-b9a9-ffcd8ae2cc01/261ee563-a4e4-4d31-ad5c-99d3e1f31c1d"
-					(reference "R8")
-					(unit 1)
-				)
-				(path "/5f9a1ba6-34f0-4af5-b9a9-ffcd8ae2cc01/b95fc682-bda1-44b2-bae0-b04d00e2d08a"
-					(reference "R2")
-					(unit 1)
-				)
-				(path "/5f9a1ba6-34f0-4af5-b9a9-ffcd8ae2cc01/da044d78-69ae-4295-a410-101a45713a38"
-					(reference "R10")
+					(reference "R5")
+					(unit 1)
+				)
+				(path "/5f9a1ba6-34f0-4af5-b9a9-ffcd8ae2cc01/b95fc682-bda1-44b2-bae0-b04d00e2d08a"
+					(reference "R6")
+					(unit 1)
+				)
+				(path "/5f9a1ba6-34f0-4af5-b9a9-ffcd8ae2cc01/da044d78-69ae-4295-a410-101a45713a38"
+					(reference "R7")
 					(unit 1)
 				)
@@
 		(dnp no)
 		(fields_autoplaced yes)
-		(property "Reference" "F4"
+		(property "Reference" "F1"
 			(at 110.49 92.71 90)
 			(effects
@@
 			(project "urban-power-dist-v2"
 				(path "/5f9a1ba6-34f0-4af5-b9a9-ffcd8ae2cc01/261ee563-a4e4-4d31-ad5c-99d3e1f31c1d"
-					(reference "F4")
-					(unit 1)
-				)
-				(path "/5f9a1ba6-34f0-4af5-b9a9-ffcd8ae2cc01/b95fc682-bda1-44b2-bae0-b04d00e2d08a"
 					(reference "F1")
 					(unit 1)
 				)
-				(path "/5f9a1ba6-34f0-4af5-b9a9-ffcd8ae2cc01/da044d78-69ae-4295-a410-101a45713a38"
-					(reference "F5")
+				(path "/5f9a1ba6-34f0-4af5-b9a9-ffcd8ae2cc01/b95fc682-bda1-44b2-bae0-b04d00e2d08a"
+					(reference "F2")
+					(unit 1)
+				)
+				(path "/5f9a1ba6-34f0-4af5-b9a9-ffcd8ae2cc01/da044d78-69ae-4295-a410-101a45713a38"
+					(reference "F3")
 					(unit 1)
 				)
@@
 		(on_board yes)
 		(dnp no)
-		(property "Reference" "D6"
+		(property "Reference" "D3"
 			(at 182.5625 90.17 0)
 			(effects
@@
 			(project "urban-power-dist-v2"
 				(path "/5f9a1ba6-34f0-4af5-b9a9-ffcd8ae2cc01/261ee563-a4e4-4d31-ad5c-99d3e1f31c1d"
-					(reference "D6")
-					(unit 1)
-				)
-				(path "/5f9a1ba6-34f0-4af5-b9a9-ffcd8ae2cc01/b95fc682-bda1-44b2-bae0-b04d00e2d08a"
 					(reference "D3")
 					(unit 1)
 				)
-				(path "/5f9a1ba6-34f0-4af5-b9a9-ffcd8ae2cc01/da044d78-69ae-4295-a410-101a45713a38"
-					(reference "D7")
+				(path "/5f9a1ba6-34f0-4af5-b9a9-ffcd8ae2cc01/b95fc682-bda1-44b2-bae0-b04d00e2d08a"
+					(reference "D4")
+					(unit 1)
+				)
+				(path "/5f9a1ba6-34f0-4af5-b9a9-ffcd8ae2cc01/da044d78-69ae-4295-a410-101a45713a38"
+					(reference "D5")
 					(unit 1)
 				)
@@
 		(dnp no)
 		(fields_autoplaced yes)
-		(property "Reference" "R9"
+		(property "Reference" "R2"
 			(at 168.91 80.01 90)
 			(effects
@@
 			(project "urban-power-dist-v2"
 				(path "/5f9a1ba6-34f0-4af5-b9a9-ffcd8ae2cc01/261ee563-a4e4-4d31-ad5c-99d3e1f31c1d"
-					(reference "R9")
-					(unit 1)
-				)
-				(path "/5f9a1ba6-34f0-4af5-b9a9-ffcd8ae2cc01/b95fc682-bda1-44b2-bae0-b04d00e2d08a"
-					(reference "R5")
-					(unit 1)
-				)
-				(path "/5f9a1ba6-34f0-4af5-b9a9-ffcd8ae2cc01/da044d78-69ae-4295-a410-101a45713a38"
-					(reference "R11")
+					(reference "R2")
+					(unit 1)
+				)
+				(path "/5f9a1ba6-34f0-4af5-b9a9-ffcd8ae2cc01/b95fc682-bda1-44b2-bae0-b04d00e2d08a"
+					(reference "R3")
+					(unit 1)
+				)
+				(path "/5f9a1ba6-34f0-4af5-b9a9-ffcd8ae2cc01/da044d78-69ae-4295-a410-101a45713a38"
+					(reference "R4")
 					(unit 1)
 				)
@@
 		(dnp no)
 		(fields_autoplaced yes)
-		(property "Reference" "J9"
+		(property "Reference" "J2"
 			(at 173.99 115.5699 0)
 			(effects
@@
 			(project "urban-power-dist-v2"
 				(path "/5f9a1ba6-34f0-4af5-b9a9-ffcd8ae2cc01/261ee563-a4e4-4d31-ad5c-99d3e1f31c1d"
-					(reference "J9")
-					(unit 1)
-				)
-				(path "/5f9a1ba6-34f0-4af5-b9a9-ffcd8ae2cc01/b95fc682-bda1-44b2-bae0-b04d00e2d08a"
-					(reference "J5")
-					(unit 1)
-				)
-				(path "/5f9a1ba6-34f0-4af5-b9a9-ffcd8ae2cc01/da044d78-69ae-4295-a410-101a45713a38"
-					(reference "J11")
-					(unit 1)
-				)
+					(reference "J2")
+					(unit 1)
+				)
+				(path "/5f9a1ba6-34f0-4af5-b9a9-ffcd8ae2cc01/b95fc682-bda1-44b2-bae0-b04d00e2d08a"
+					(reference "J3")
+					(unit 1)
+				)
+				(path "/5f9a1ba6-34f0-4af5-b9a9-ffcd8ae2cc01/da044d78-69ae-4295-a410-101a45713a38"
+					(reference "J4")
+					(unit 1)
+				)

Commit message: layout DRC fixes
Parts:
- J2: footprint ATF13-2P-BM03:ATF132PBM03 -> connector footprint:ATF132PBM03
Changed lines of the file:
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@@
 			)
 		)
-		(property "Footprint" "ATF13-2P-BM03:ATF132PBM03"
+		(property "Footprint" "connector footprint:ATF132PBM03"
 			(at 172.72 115.57 0)
 			(effects
