File: urban-power-dist-v2.kicad_pcb (KiCad board)
At the start: 2 copper layers, 110 x 110 mm, 27 parts, among them J1 12V_IN, J2 OUT, J3 OUT, J4 OUT, J5 TEST_PT, J6 TEST_PT, J7 TEST_PT

Commit message: final pcb edits
Other:
- board text added: "[BOARD NAME HERE] Aaron Li, Samantha Sheh SEMA 2026"
- board text removed: "FRONT LED"
- board text removed: "REAR LED"
- board text removed: "TEL LED"
- board text removed: "[BOARD NAME HERE] Aaron L, Samantha S SEMA 2026"
Changed lines of the file:
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@@
 			(at 0 -4.15 0)
 			(layer "F.SilkS")
+			(hide yes)
 			(effects
 				(font
@@
 			(at 0 -4.15 0)
 			(layer "F.SilkS")
+			(hide yes)
 			(effects
 				(font
@@
 			(at 0 -4.15 0)
 			(layer "F.SilkS")
+			(hide yes)
 			(effects
 				(font
@@
 			(at 0 -4.15 0)
 			(layer "F.SilkS")
+			(hide yes)
 			(effects
 				(font
@@
 		)
 	)
-	(gr_text "[BOARD NAME HERE]\nAaron L, Samantha S\nSEMA 2026"
+	(gr_text "[BOARD NAME HERE]\nAaron Li, Samantha Sheh\nSEMA 2026"
 		(at 155 115 0)
 		(layer "F.SilkS")
@@
 		)
 	)
-	(gr_text "TEL\nLED"
-		(at 160.47375 64.5 0)
+	(gr_text "TEL"
+		(at 160.47375 65 0)
 		(layer "F.SilkS")
 		(effects
@@
 		)
 	)
-	(gr_text "REAR\nLED"
-		(at 195.5 110.47375 0)
+	(gr_text "REAR"
+		(at 196 110.47375 0)
 		(layer "F.SilkS")
 		(effects
@@
 		)
 	)
-	(gr_text "FRONT\nLED"
+	(gr_text "FRONT"
 		(at 111.5 92.5 0)
 		(layer "F.SilkS")

Commit message: shuriken
Other:
- board text added: "Shuriken Aaron Li, Samantha Sheh SEMA 2026"
- board text removed: "[BOARD NAME HERE] Aaron Li, Samantha Sheh SEMA 2026"
Changed lines of the file:
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@@
 		)
 	)
-	(gr_text "[BOARD NAME HERE]\nAaron Li, Samantha Sheh\nSEMA 2026"
+	(gr_text "Shuriken\nAaron Li, Samantha Sheh\nSEMA 2026"
 		(at 155 115 0)
 		(layer "F.SilkS")
@@
 	)
 	(gr_text "FRONT"
-		(at 111.5 92.5 0)
-		(layer "F.SilkS")
-		(effects
+		(at 113.5 99.75 0)
+		(layer "F.SilkS")
+		(effects
